Commit message: modify caster size, and request speed

File: assignment_2/src/my_robot/urdf/my_robot.xacro (robot description, xacro)
@@ -34,5 +34,5 @@
       <origin xyz="-0.15 0 -0.075" rpy=" 0 0 0"/>
       <geometry>
-        <sphere radius="0.07499"/>
+        <sphere radius="0.07495"/>
       </geometry>
     </collision>
@@ -46,5 +46,5 @@
       <origin xyz="0.15 0 -0.075" rpy=" 0 0 0"/>
       <geometry>
-        <sphere radius="0.07499"/>
+        <sphere radius="0.07495"/>
       </geometry>
     </collision>

Commit message: make changes related to review

File: assignment_2/src/my_robot/urdf/my_robot.xacro (robot description, xacro)
@@ -191,14 +191,14 @@
   </joint>
   <gazebo reference="left_wheel">
-    <material>Gazebo/Blue</material>
+    <material>Gazebo/Black</material>
   </gazebo>
   <gazebo reference="right_wheel">
-    <material>Gazebo/Blue</material>
+    <material>Gazebo/Black</material>
   </gazebo>
   <gazebo reference="chassis">
+    <material>Gazebo/Purple</material>
+  </gazebo>
+  <gazebo reference="camera">
     <material>Gazebo/Green</material>
   </gazebo>
-  <gazebo reference="camera">
-    <material>Gazebo/Red</material>
-  </gazebo>
 </robot>
