Commit message: add markers and pickup

File: src/my_robot/urdf/mapping_robot.xacro (robot description, xacro)
@@ -11,5 +11,5 @@
     <pose>0 0 0.1 0 0 0</pose>
     <inertial>
-      <mass value="15.0"/>
+      <mass value="12.0"/>
       <origin xyz="0.0 0 0.0" rpy=" 0 0 0"/>
       <inertia
@@ -22,5 +22,5 @@
       <origin xyz="0 0 0.0" rpy=" 0 0 0"/>
       <geometry>
-        <box size=".5 .4 .15"/>
+        <box size=".4 .3 .1"/>
       </geometry>
     </collision>
@@ -28,29 +28,29 @@
       <origin xyz="0 0 0.0" rpy=" 0 0 0"/>
       <geometry>
-        <box size=".5 .4 .15"/>
+        <box size=".4 .3 .1"/>
       </geometry>
     </visual>
     <collision name='back_caster_collision'>
-      <origin xyz="-0.15 0 -0.075" rpy=" 0 0 0"/>
-      <geometry>
-        <sphere radius="0.07495"/>
+      <origin xyz="-0.15 0 -0.05" rpy=" 0 0 0"/>
+      <geometry>
+        <sphere radius="0.0499"/>
       </geometry>
     </collision>
     <visual name='back_caster_visual'>
-      <origin xyz="-0.15 0 -0.075" rpy=" 0 0 0"/>
-      <geometry>
-        <sphere radius="0.075"/>
+      <origin xyz="-0.15 0 -0.05" rpy=" 0 0 0"/>
+      <geometry>
+        <sphere radius="0.05"/>
       </geometry>
     </visual>
     <collision name='front_caster_collision'>
-      <origin xyz="0.15 0 -0.075" rpy=" 0 0 0"/>
-      <geometry>
-        <sphere radius="0.07495"/>
+      <origin xyz="0.15 0 -0.05" rpy=" 0 0 0"/>
+      <geometry>
+        <sphere radius="0.0499"/>
       </geometry>
     </collision>
     <visual name='front_caster_visual'>
-      <origin xyz="0.15 0 -0.075" rpy=" 0 0 0"/>
-      <geometry>
-        <sphere radius="0.075"/>
+      <origin xyz="0.15 0 -0.05" rpy=" 0 0 0"/>
+      <geometry>
+        <sphere radius="0.05"/>
       </geometry>
     </visual>
@@ -70,5 +70,5 @@
   <link name='left_wheel'>
     <inertial>
-      <mass value="5.0"/>
+      <mass value="2.0"/>
       <origin xyz="0.0 0 0.0" rpy="0 1.5707 1.5707"/>
       <inertia
@@ -81,5 +81,5 @@
       <origin xyz="0 0 0.0" rpy="0 1.5707 1.5707"/>
       <geometry>
-        <cylinder radius="0.15" length="0.05"/>
+        <cylinder radius="0.1" length="0.05"/>
       </geometry>
     </collision>
@@ -87,5 +87,5 @@
       <origin xyz="0 0 0.0" rpy="0 1.5707 1.5707"/>
       <geometry>
-        <cylinder radius="0.15" length="0.05"/>
+        <cylinder radius="0.1" length="0.05"/>
       </geometry>
     </visual>
@@ -93,5 +93,5 @@
   <link name='right_wheel'>
     <inertial>
-      <mass value="5.0"/>
+      <mass value="2.0"/>
       <origin xyz="0.0 0 0.0" rpy="0 1.5707 1.5707"/>
       <inertia
@@ -104,5 +104,5 @@
       <origin xyz="0 0 0.0" rpy="0 1.5707 1.5707"/>
       <geometry>
-        <cylinder radius="0.15" length="0.05"/>
+        <cylinder radius="0.1" length="0.05"/>
       </geometry>
     </collision>
@@ -110,5 +110,5 @@
       <origin xyz="0 0 0.0" rpy="0 1.5707 1.5707"/>
       <geometry>
-        <cylinder radius="0.15" length="0.05"/>
+        <cylinder radius="0.1" length="0.05"/>
       </geometry>
     </visual>
@@ -141,5 +141,5 @@
     <origin xyz="0 0 0" rpy="0 0 0"/>
     <inertial>
-      <mass value="0.1"/>
+      <mass value="1e-5"/>
       <origin xyz="0.05 0.05 0.05"/>
       <inertia
@@ -169,5 +169,5 @@
   <link name="camera_link_optical"/>
   <joint type="continuous" name="left_wheel_hinge">
-    <origin xyz="0 0.25 0" rpy="0 0 0"/>
+    <origin xyz="0 0.2 0" rpy="0 0 0"/>
     <child link="left_wheel"/>
     <parent link="chassis"/>
@@ -177,5 +177,5 @@
   </joint>
   <joint type="continuous" name="right_wheel_hinge">
-    <origin xyz="0 -0.25 0" rpy="0 0 0"/>
+    <origin xyz="0 -0.2 0" rpy="0 0 0"/>
     <child link="right_wheel"/>
     <parent link="chassis"/>
@@ -198,9 +198,17 @@
   <gazebo reference="left_wheel">
     <material>Gazebo/Black</material>
+	<mu1>0.3</mu1>
+	<mu2>0.3</mu2>
+	<minDepth>0.01</minDepth>
   </gazebo>
   <gazebo reference="right_wheel">
     <material>Gazebo/Black</material>
+	<mu1>0.3</mu1>
+	<mu2>0.3</mu2>
+	<minDepth>0.01</minDepth>
   </gazebo>
   <gazebo reference="chassis">
+    <mu1>0.0</mu1>
+    <mu2>0.0</mu2>
     <material>Gazebo/Purple</material>
   </gazebo>
